File: Circuit/Circuit.kicad_pcb (KiCad board)
At the start: 2 copper layers, 182.9 x 203.2 mm, 103 parts, among them J1 Conn_01x02_Male, SW1 SW_Push, SW10 SW_Push, SW11 SW_Push, SW12 SW_Push, SW13 SW_Push, SW14 SW_Push, SW15 SW_Push, SW16 SW_Push, SW17 SW_Push, SW2 SW_Push, SW3 SW_Push, SW4 SW_Push, SW5 SW_Push, SW6 SW_Push, SW7 SW_Push, SW8 SW_Push, U1 AD9833, U2 LM386, U3 MAX7219

Commit message: Added more traces, added all footprints, and made minor corrections to schematic.
Parts:
- added BT1: Battery_Cell, Connector_JST:JST_EH_B2B-EH-A_1x02_P2.50mm_Vertical, F.Cu at (174.0, -83.8)
- added C1: 100nF, Capacitor_THT:C_Disc_D4.3mm_W1.9mm_P5.00mm, F.Cu at (132.1, -78.8)
- added C2: 100nF, Capacitor_THT:C_Disc_D4.3mm_W1.9mm_P5.00mm, F.Cu at (29.2, -48.3)
- added C3: 470μF, Capacitor_THT:CP_Radial_D14.0mm_P7.50mm, F.Cu at (174.0, -72.4)
- added C4: 100nF, Capacitor_THT:C_Disc_D4.3mm_W1.9mm_P5.00mm, F.Cu at (169.6, -31.8)
- added C5: 100nF, Capacitor_THT:C_Disc_D4.3mm_W1.9mm_P5.00mm, F.Cu at (185.4, -40.7)
- added C6: 470μF, Capacitor_THT:CP_Radial_D14.0mm_P7.50mm, F.Cu at (182.9, -68.6)
- added C7: 100nF, Capacitor_THT:C_Disc_D4.3mm_W1.9mm_P5.00mm, F.Cu at (160.0, -71.0)
- added J10: SPKR, Connector_PinHeader_2.54mm:PinHeader_1x02_P2.54mm_Vertical, F.Cu at (188.0, -78.7)
- added J2: 3V3, Connector_PinHeader_2.54mm:PinHeader_1x01_P2.54mm_Vertical, F.Cu at (63.5, -67.8)
- added J3: LM386 VCC, Connector_PinHeader_2.54mm:PinHeader_1x01_P2.54mm_Vertical, F.Cu at (174.0, -62.2)
- added J4: BYPASS, Connector_PinHeader_2.54mm:PinHeader_1x01_P2.54mm_Vertical, F.Cu at (161.3, -55.9)
- added J5: LM386 OUT, Connector_PinHeader_2.54mm:PinHeader_1x01_P2.54mm_Vertical, F.Cu at (176.5, -62.2)
- added J6: AD9833 OUT, Connector_PinHeader_2.54mm:PinHeader_1x01_P2.54mm_Vertical, F.Cu at (159.4, -31.8)
- added J7: LM386 IN, Connector_PinHeader_2.54mm:PinHeader_1x03_P2.54mm_Vertical, F.Cu at (174.0, -47.0)
- added J8: GAIN 1, Connector_PinHeader_2.54mm:PinHeader_1x01_P2.54mm_Vertical, F.Cu at (161.3, -53.3)
- added J9: GAIN 8, Connector_PinHeader_2.54mm:PinHeader_1x01_P2.54mm_Vertical, F.Cu at (161.3, -58.4)
- added LS1: 8Ω, Connector_JST:JST_EH_B2B-EH-A_1x02_P2.50mm_Vertical, F.Cu at (187.9, -83.8)
- added R1: 10K, Resistor_THT:R_Axial_DIN0207_L6.3mm_D2.5mm_P7.62mm_Horizontal, F.Cu at (24.1, -44.5)
- added U4: MAX7219, Package_DIP:DIP-24_W7.62mm_LongPads, F.Cu at (16.5, -30.5)
- D1, D10, D11, D12, D13, D14, D15, D16, D2, D3, D4, D5, D6, D7, D8, D9: footprint Diode_SMD:D_SC-80_HandSoldering -> Diode_SMD:D_SMB_Handsoldering
- J1: value Conn_01x02_Male -> VIN; footprint Connector_PinHeader_2.54mm:PinHeader_1x02_P2.54mm_Vertical -> Connector_PinHeader_2.54mm:PinHeader_1x01_P2.54mm_Vertical
- R2: value 10K -> 10
- RV1: value R_POT -> 20K; moved to F.Cu
- U1: value AD9833 -> MicroSDSparkfun; footprint Connector_PinHeader_2.54mm:PinHeader_1x07_P2.54mm_Vertical -> Connector_PinHeader_2.54mm:PinHeader_1x07_P2.54mm_Horizontal
- U2: value LM386 -> AD9833; footprint Package_DIP:DIP-8_W7.62mm_Socket_LongPads -> Connector_PinHeader_2.54mm:PinHeader_1x07_P2.54mm_Vertical; moved to F.Cu
- U3: value MAX7219 -> LM386; footprint Package_DIP:DIP-24_W7.62mm_LongPads -> Package_DIP:DIP-8_W7.62mm_Socket_LongPads
- moved J1 273.5 mm to (63.5, -57.1), turned to 0 degrees
- moved A1 144.4 mm to (73.7, -74.9)
- moved U3 144.1 mm to (168.9, -50.8), turned to 90 degrees
- moved D11 136.8 mm to (130.3, 147.3)
- moved D14 136.8 mm to (168.4, 147.3)
- moved D16 136.8 mm to (187.5, 147.3)
- moved D2 136.8 mm to (35.1, 147.3)
- moved D20 136.8 mm to (47.6, 161.3)
- moved D23 136.8 mm to (85.7, 161.3)
- moved D25 136.8 mm to (104.8, 161.3)
- moved D32 136.8 mm to (181.0, 161.3)
- moved D4 136.8 mm to (54.1, 147.3)
- moved D8 136.8 mm to (92.2, 147.3)
- moved SW10 136.8 mm to (108.6, 151.1)
- moved D1 136.8 mm to (25.6, 166.4)
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- renumbered SW11 to SW10, SW12 to SW11, SW13 to SW12, SW14 to SW13, SW15 to SW14, SW16 to SW15, SW17 to SW16, SW10 to SW9
Connections:
- A1 pad 23: (no net) -> /SS_SDCARD
- A1 pad 27: (no net) -> /SPI_MISO
- A1 pad 29: (no net) -> GND
- A1 pad 4: (no net) -> Net-(A1-Pad4)
- A1 pad 5: (no net) -> VCC
- A1 pad 7: (no net) -> GND
- A1 pad 8: VCC -> Net-(A1-Pad8)
- A1 pad 9: (no net) -> /SDCARD_CD
- J1 pad 1: GND -> Net-(A1-Pad8)
- R2 pad 1: VCC -> Net-(C7-Pad1)
- R2 pad 2: Net-(R2-Pad2) -> GND
- RV1 pad 1: Net-(RV1-Pad1) -> Net-(J6-Pad1)
- RV1 pad 2: (no net) -> Net-(C5-Pad2)
- U1 pad 1: (no net) -> VCC
- U1 pad 2: (no net) -> /SS_SDCARD
- U1 pad 5: /SS_AD9837 -> /SPI_MISO
- U1 pad 6: (no net) -> /SDCARD_CD
- U1 pad 7: Net-(RV1-Pad1) -> GND
- U2 pad 1: (no net) -> VCC
- U2 pad 3: (no net) -> /SPI_MOSI
- U2 pad 4: GND -> /SPI_SCK
- U2 pad 5: (no net) -> /SS_AD9837
- U2 pad 6: Net-(J1-Pad2) -> GND
- U2 pad 7: (no net) -> Net-(J6-Pad1)
- U3 pad 1: /SPI_MOSI -> Net-(J8-Pad1)
- U3 pad 2: /DIG_0 -> Net-(J7-Pad2)
- U3 pad 3: /DIG_4 -> Net-(C5-Pad1)
- U3 pad 5: /DIG_6 -> Net-(C6-Pad1)
- U3 pad 6: /DIG_2 -> +9V
- U3 pad 7: /DIG_3 -> Net-(J4-Pad1)
- U3 pad 8: /DIG_7 -> Net-(J9-Pad1)
Routing:
- net /SW_COL_2: track 0.00 -> 391.6 mm, vias 0 -> 6
- net /SW_COL_3: track 0.00 -> 374.9 mm, vias 0 -> 4
- net /SW_COL_0: track 0.00 -> 371.8 mm, vias 0 -> 4
- net /SW_COL_1: track 67.8 -> 375.2 mm, vias 2 -> 4
- net Net-(D25-Pad2): track 124.1 -> 412.8 mm, vias 0 -> 1
- net /SW_ROW_3: track 38.1 -> 278.9 mm, vias 0 -> 2
- net /SW_ROW_0: track 85.2 -> 323.3 mm, vias 0 -> 2
- net Net-(D41-Pad2): track 136.0 -> 373.7 mm, vias 2 -> 3
- net Net-(D17-Pad2): track 120.5 -> 341.7 mm, vias 1 -> 2
- net /SW_ROW_2: track 38.1 -> 258.2 mm, vias 0 -> 1
- net /SW_ROW_1: track 82.5 -> 279.6 mm, vias 0 -> 2
- net Net-(D57-Pad2): track 100.3 -> 284.8 mm, vias 0 -> 2
- net Net-(D33-Pad2): track 138.5 -> 301.9 mm
- net Net-(D49-Pad2): track 100.3 -> 246.1 mm, vias 0 -> 1
- net /SPI_MOSI: track 0.00 -> 134.9 mm
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- added copper zone on B.Cu, net GND
- added copper zone on F.Cu, net GND
Other:
- board size 182.9 x 203.2 mm -> 182.9 x 271.8 mm
- net class Power added: clearance 0.4, trace_width 0.5, via_dia 1, via_drill 0.6

Commit message: Upload final version of Schematic and board layout.
Parts:
- removed the C7 at (160.0, -71.0)
- removed the J6 at (159.4, -31.8)
- removed the J7 at (174.0, -47.0)
- added C2: 100nF, Capacitor_THT:C_Disc_D4.3mm_W1.9mm_P5.00mm, F.Cu at (160.7, -64.1)
- added C8: 100nF, Capacitor_THT:C_Disc_D4.3mm_W1.9mm_P5.00mm, F.Cu at (180.3, -27.9)
- added J10: LM386 IN, Connector_PinHeader_2.54mm:PinHeader_1x03_P2.54mm_Vertical, F.Cu at (174.0, -47.0)
- added J3: AREF, Connector_PinHeader_2.54mm:PinHeader_1x01_P2.54mm_Vertical, F.Cu at (128.3, -78.7)
- added J4: Analog Breakout, Connector_PinHeader_2.54mm:PinHeader_1x05_P2.54mm_Vertical, F.Cu at (67.3, -49.5)
- added J5: SPI (MOSI, MISO, SCK), Connector_PinHeader_2.54mm:PinHeader_1x03_P2.54mm_Vertical, F.Cu at (128.3, -68.6)
- added J9: AD9833 OUT, Connector_PinHeader_2.54mm:PinHeader_1x01_P2.54mm_Vertical, F.Cu at (167.6, -28.6)
- added JP1: Jumper, Connector_PinHeader_2.54mm:PinHeader_1x02_P2.54mm_Vertical, F.Cu at (186.7, -54.0)
- J1: value VIN -> POWER; footprint Connector_PinHeader_2.54mm:PinHeader_1x01_P2.54mm_Vertical -> Connector_PinHeader_2.54mm:PinHeader_1x04_P2.54mm_Vertical
- J2: value 3V3 -> RESET
- J6: renamed from J3; value LM386 VCC -> 9V
- moved R2 49.8 mm to (176.5, -27.9)
- moved U2 31.9 mm to (142.9, -38.1), turned to 90 degrees
- moved C4 24.0 mm to (147.9, -41.9), turned to 180 degrees
- moved C6 11.5 mm to (174.0, -41.9), turned to 0 degrees
- moved J2 9.22 mm to (67.3, -76.2)
- moved J1 8.52 mm to (67.3, -64.8), turned to 180 degrees
- moved RV1 5.68 mm to (188.0, -39.4)
- moved U1 1.91 mm to (138.4, -76.2)
- moved C1 1.27 mm to (133.3, -78.8)
- renumbered C2 to C5, C5 to C6, C6 to C7, J8 to J11, J9 to J12, J10 to J13, J4 to J7, J5 to J8
Connections:
- A1 pad 10: (no net) -> Net-(A1-Pad10)
- A1 pad 11: (no net) -> Net-(A1-Pad11)
- A1 pad 12: (no net) -> Net-(A1-Pad12)
- A1 pad 13: (no net) -> Net-(A1-Pad13)
- A1 pad 14: (no net) -> Net-(A1-Pad14)
- A1 pad 3: (no net) -> Net-(A1-Pad3)
- A1 pad 30: (no net) -> Net-(A1-Pad30)
- J1 pad 1: Net-(A1-Pad8) -> VCC
- J2 pad 1: Net-(A1-Pad4) -> Net-(A1-Pad3)
Routing:
- net VCC: track 72.4 -> 333.6 mm, vias 0 -> 2
- net /SS_MAX7219: track 0.55 -> 98.6 mm, vias 0 -> 1
- net /SDCARD_CD: track 0.00 -> 95.6 mm
- net /SPI_SCK: track 92.6 -> 157.8 mm
- net /SPI_MOSI: track 134.9 -> 198.5 mm, vias 0 -> 1
- net /SS_SDCARD: track 0.00 -> 58.3 mm
- net /SS_AD9837: track 0.00 -> 53.2 mm
- net Net-(J9-Pad1): track 3.81 -> 43.8 mm
- net /SPI_MISO: track 0.00 -> 28.9 mm
- net Net-(C8-Pad2): track 0.00 -> 23.7 mm
- net Net-(C7-Pad2): track 0.00 -> 16.3 mm
- net GND: track 0.00 -> 14.0 mm
- net +9V: track 25.4 -> 34.4 mm
- net Net-(A1-Pad3): track 0.00 -> 8.98 mm
- net Net-(C6-Pad2): track 0.00 -> 8.97 mm
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Other:
- board text added: "+"
- board text added: "-"
- board text added: "A1 A2 A3 A4 A5"
- board text added: "Ebrahimi Frieda Indictor Manrique Xu"
- board text added: "GND VIN 3V3 5V"
- board text added: "JLCJLCJLCJLC"
